File: v6/ENV6_DemoBoard_1/MCU.kicad_sch (KiCad schematic)
At the start: 42 parts, among them J401 Pico Debugger (SWD), J402 Conn_01x04_Pin, U401 RP2354B, U402 Pi-Radio, U403 W25Q16JVUXIQ, Y401 KX7_QRZ

Commit message: SPartan7Board and new Symbol and Footprint
Parts:
- C401, C402, C403, C404, C405, C406, C407, C408, C409, C410, C414, C415, C416: value 100n -> 1u
- C411, C412: value 10u -> 1u
Connections:
- net CFG_DONE renamed FPGA_CFG_3
- net CFG_Extra renamed FPGA_CFG_5
- net CFG_FAILED_N renamed FPGA_CFG_4
- net FPGA_RST renamed FPGA_CFG_1
- net POR_EN renamed FPGA_CFG_2
Changed lines of the file:
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@@
 		)
 	)
+	(global_label "FPGA_CFG_2"
+		(shape bidirectional)
+		(at 137.16 109.22 0)
+		(fields_autoplaced yes)
+		(effects
+			(font
+				(size 1.27 1.27)
+			)
+			(justify left)
+		)
+		(property "Intersheetrefs" "${INTERSHEET_REFS}"
+			(at 152.747 109.22 0)
+			(hide yes)
+			(show_name no)
+			(do_not_autoplace no)
+			(effects
+				(font
+					(size 1.27 1.27)
+				)
+				(justify left)
+			)
+		)
+	)
 	(global_label "JTAG_TMS_GP19"
 		(shape bidirectional)
@@
 		)
 	)
+	(global_label "FPGA_CFG_4"
+		(shape bidirectional)
+		(at 137.16 133.35 0)
+		(fields_autoplaced yes)
+		(effects
+			(font
+				(size 1.27 1.27)
+			)
+			(justify left)
+		)
+		(property "Intersheetrefs" "${INTERSHEET_REFS}"
+			(at 152.747 133.35 0)
+			(hide yes)
+			(show_name no)
+			(do_not_autoplace no)
+			(effects
+				(font
+					(size 1.27 1.27)
+				)
+				(justify left)
+			)
+		)
+	)
 	(global_label "GP38{slash}SPI0_SCK"
 		(shape bidirectional)
@@
 		)
 	)
-	(global_label "GP14{slash}SPI1_SCK"
+	(global_label "FPGA_CFG_3"
 		(shape bidirectional)
-		(at 138.43 88.9 0)
+		(at 137.16 111.76 0)
 		(fields_autoplaced yes)
 		(effects
@@
 		)
 		(property "Intersheetrefs" "${INTERSHEET_REFS}"
-			(at 157.8269 88.9 0)
+			(at 152.747 111.76 0)
 			(hide yes)
 			(show_name no)
@@
 		)
 	)
-	(global_label "ADC_Detect2"
+	(global_label "GP14{slash}SPI1_SCK"
 		(shape bidirectional)
-		(at 137.16 167.64 0)
+		(at 138.43 88.9 0)
 		(fields_autoplaced yes)
 		(effects
@@
 		)
 		(property "Intersheetrefs" "${INTERSHEET_REFS}"
-			(at 153.0494 167.64 0)
+			(at 157.8269 88.9 0)
 			(hide yes)
 			(show_name no)
@@
 		)
 	)
-	(global_label "GP1{slash}I2C0_SCL"
+	(global_label "ADC_Detect2"
 		(shape bidirectional)
-		(at 137.16 53.34 0)
-		(fields_autoplaced yes)
-		(effects
-			(font
-				(size 1.27 1.27)
-			)
-			(justify left)
-		)
-		(property "Intersheetrefs" "${INTERSHEET_REFS}"
-			(at 155.1055 53.34 0)
-			(hide yes)
-			(show_name no)
-			(do_not_autoplace no)
-			(effects
-				(font
-					(size 1.27 1.27)
-				)
-				(justify left)
-			)
-		)
-	)
-	(global_label "CFG_DONE"
-		(shape input)
-		(at 137.16 111.76 0)
-		(fields_autoplaced yes)
-		(effects
-			(font
-				(size 1.27 1.27)
-			)
-			(justify left)
-		)
-		(property "Intersheetrefs" "${INTERSHEET_REFS}"
-			(at 149.8214 111.76 0)
-			(hide yes)
-			(show_name no)
-			(do_not_autoplace no)
-			(effects
-				(font
-					(size 1.27 1.27)
-				)
-				(justify left)
-			)
-		)
-	)
-	(global_label "POR_EN"
-		(shape output)
-		(at 137.16 109.22 0)
+		(at 137.16 167.64 0)
 		(fields_autoplaced yes)
 		(effects
@@
 		)
 		(property "Intersheetrefs" "${INTERSHEET_REFS}"
-			(at 147.4628 109.22 0)
+			(at 153.0494 167.64 0)
 			(hide yes)
 			(show_name no)
@@
 		)
 	)
-	(global_label "CFG_Extra"
-		(shape output)
-		(at 137.16 128.27 0)
+	(global_label "GP1{slash}I2C0_SCL"
+		(shape bidirectional)
+		(at 137.16 53.34 0)
 		(fields_autoplaced yes)
 		(effects
@@
 		)
 		(property "Intersheetrefs" "${INTERSHEET_REFS}"
-			(at 149.5794 128.27 0)
+			(at 155.1055 53.34 0)
 			(hide yes)
 			(show_name no)
@@
 		)
 	)
-	(global_label "GP0{slash}I2C0_SDA"
+	(global_label "FPGA_CFG_5"
 		(shape bidirectional)
-		(at 124.46 33.02 180)
+		(at 137.16 128.27 0)
 		(fields_autoplaced yes)
 		(effects
@@
 				(size 1.27 1.27)
 			)
-			(justify right)
+			(justify left)
 		)
 		(property "Intersheetrefs" "${INTERSHEET_REFS}"
-			(at 106.454 33.02 0)
+			(at 152.747 128.27 0)
 			(hide yes)
 			(show_name no)
@@
 					(size 1.27 1.27)
 				)
-				(justify right)
+				(justify left)
 			)
 		)
 	)
-	(global_label "LP_nRST"
+	(global_label "GP0{slash}I2C0_SDA"
 		(shape bidirectional)
-		(at 137.16 55.88 0)
+		(at 124.46 33.02 180)
 		(fields_autoplaced yes)
 		(effects
@@
 				(size 1.27 1.27)
 			)
-			(justify left)
+			(justify right)
 		)
 		(property "Intersheetrefs" "${INTERSHEET_REFS}"
-			(at 149.1183 55.88 0)
+			(at 106.454 33.02 0)
 			(hide yes)
 			(show_name no)
@@
 					(size 1.27 1.27)
 				)
-				(justify left)
+				(justify right)
 			)
 		)
 	)
-	(global_label "JTAG_TDI_GP16"
+	(global_label "LP_nRST"
 		(shape bidirectional)
-		(at 137.16 96.52 0)
+		(at 137.16 55.88 0)
 		(fields_autoplaced yes)
 		(effects
@@
 		)
 		(property "Intersheetrefs" "${INTERSHEET_REFS}"
-			(at 155.2869 96.52 0)
+			(at 149.1183 55.88 0)
 			(hide yes)
 			(show_name no)
@@
 		)
 	)
-	(global_label "JTAG_TCK_GP18"
+	(global_label "JTAG_TDI_GP16"
 		(shape bidirectional)
-		(at 137.16 101.6 0)
+		(at 137.16 96.52 0)
 		(fields_autoplaced yes)
 		(effects
@@
 		)
 		(property "Intersheetrefs" "${INTERSHEET_REFS}"
-			(at 155.9521 101.6 0)
+			(at 155.2869 96.52 0)
 			(hide yes)
 			(show_name no)
@@
 		)
 	)
-	(global_label "CFG_FAILED_N"
-		(shape input)
-		(at 137.16 133.35 0)
+	(global_label "JTAG_TCK_GP18"
+		(shape bidirectional)
+		(at 137.16 101.6 0)
 		(fields_autoplaced yes)
 		(effects
@@
 		)
 		(property "Intersheetrefs" "${INTERSHEET_REFS}"
-			(at 153.2686 133.35 0)
+			(at 155.9521 101.6 0)
 			(hide yes)
 			(show_name no)
@@
 		)
 	)
-	(global_label "FPGA_RST"
+	(global_label "FPGA_CFG_1"
 		(shape bidirectional)
 		(at 137.16 106.68 0)
@@
 		)
 		(property "Intersheetrefs" "${INTERSHEET_REFS}"
-			(at 150.3884 106.68 0)
+			(at 152.747 106.68 0)
 			(hide yes)
 			(show_name no)
@@
 			)
 		)
-		(property "Value" "100n"
+		(property "Value" "1u"
 			(at 57.658 59.69 0)
 			(show_name no)
@@
 			)
 		)
-		(property "Value" "100n"
+		(property "Value" "1u"
 			(at 213.36 146.0499 0)
 			(show_name no)
@@
 			)
 		)
-		(property "Value" "100n"
+		(property "Value" "1u"
 			(at 91.948 59.69 0)
 			(show_name no)
@@
 			)
 		)
-		(property "Value" "100n"
+		(property "Value" "1u"
 			(at 80.518 59.69 0)
 			(show_name no)
@@
 			)
 		)
-		(property "Value" "100n"
+		(property "Value" "1u"
 			(at 34.798 59.69 0)
 			(show_name no)
@@
 			)
 		)
-		(property "Value" "10u"
+		(property "Value" "1u"
 			(at 80.518 87.63 0)
 			(show_name no)
@@
 			)
 		)
-		(property "Value" "100n"
+		(property "Value" "1u"
 			(at 91.948 45.72 0)
 			(show_name no)
@@
 			)
 		)
-		(property "Value" "100n"
+		(property "Value" "1u"
 			(at 80.518 45.72 0)
 			(show_name no)
@@
 			)
 		)
-		(property "Value" "100n"
+		(property "Value" "1u"
 			(at 23.368 59.69 0)
 			(show_name no)
@@
 			)
 		)
-		(property "Value" "100n"
+		(property "Value" "1u"
 			(at 69.088 59.69 0)
 			(show_name no)
@@
 			)
 		)
-		(property "Value" "100n"
+		(property "Value" "1u"
 			(at 69.088 45.72 0)
 			(show_name no)
@@
 			)
 		)
-		(property "Value" "10u"
+		(property "Value" "1u"
 			(at 80.518 73.66 0)
 			(show_name no)
@@
 			)
 		)
-		(property "Value" "100n"
+		(property "Value" "1u"
 			(at 22.733 132.08 0)
 			(show_name no)
@@
 			)
 		)
-		(property "Value" "100n"
+		(property "Value" "1u"
 			(at 46.228 59.69 0)
 			(show_name no)
@@
 			)
 		)
-		(property "Value" "100n"
+		(property "Value" "1u"
 			(at 200.66 146.0499 0)
 			(show_name no)

Commit message: Fix small errors for the design
Parts:
- renumbered C404 to C401, C414 to C402, C405 to C403, C406 to C404, C407 to C405, C401 to C406, C408 to C407, C402 to C408, C411 to C410, C412 to C411, C417 to C412, C403 to C413, C410 to C414, C418 to C415, C413 to C416, C415 to C417, C416 to C418, R410 to R401, R411 to R402, R408 to R403, R407 to R404, R409 to R405, R403 to R406, R404 to R407, R401 to R408, R402 to R409, R405 to R410, R406 to R411, S403 to S401, S401 to S402, S402 to S403, U403 to U401, U401 to U402, U402 to U403
