File: v6/ENV6_DemoBoard_1/Power.kicad_sch (KiCad schematic)
At the start: 38 parts, among them IC301 LP873300RHDTQ1, U301 BQ25188, U302 TPSM8310x

Commit message: SPartan7Board and new Symbol and Footprint
Parts:
- C301, C304, C306: value 100n -> 1u
- C302, C303, C305, C307, C308, C309, C310, C311, C312, C313, C314, C315, C316, C317, C318, C319, C320, C321, C322: value 10u -> 1u
- L301, L302: value 0.47uH -> 0.47u
Changed lines of the file:
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@@
 			)
 		)
-		(property "Value" "100n"
+		(property "Value" "1u"
 			(at 91.948 43.18 0)
 			(show_name no)
@@
 			)
 		)
-		(property "Value" "10u"
+		(property "Value" "1u"
 			(at 67.818 115.57 0)
 			(show_name no)
@@
 			)
 		)
-		(property "Value" "10u"
+		(property "Value" "1u"
 			(at 123.698 146.05 0)
 			(show_name no)
@@
 			)
 		)
-		(property "Value" "10u"
+		(property "Value" "1u"
 			(at 57.658 115.57 0)
 			(show_name no)
@@
 			)
 		)
-		(property "Value" "10u"
+		(property "Value" "1u"
 			(at 204.978 48.26 0)
 			(show_name no)
@@
 			)
 		)
-		(property "Value" "10u"
+		(property "Value" "1u"
 			(at 204.978 63.5 0)
 			(show_name no)
@@
 			)
 		)
-		(property "Value" "0.47uH"
+		(property "Value" "0.47u"
 			(at 120.65 113.538 90)
 			(show_name no)
@@
 			)
 		)
-		(property "Value" "10u"
+		(property "Value" "1u"
 			(at 67.818 130.81 0)
 			(show_name no)
@@
 			)
 		)
-		(property "Value" "10u"
+		(property "Value" "1u"
 			(at 207.518 125.73 0)
 			(show_name no)
@@
 			)
 		)
-		(property "Value" "100n"
+		(property "Value" "1u"
 			(at 217.678 48.26 0)
 			(show_name no)
@@
 			)
 		)
-		(property "Value" "10u"
+		(property "Value" "1u"
 			(at 67.818 146.05 0)
 			(show_name no)
@@
 			)
 		)
-		(property "Value" "10u"
+		(property "Value" "1u"
 			(at 123.698 130.81 0)
 			(show_name no)
@@
 			)
 		)
-		(property "Value" "10u"
+		(property "Value" "1u"
 			(at 204.978 34.29 0)
 			(show_name no)
@@
 			)
 		)
-		(property "Value" "10u"
+		(property "Value" "1u"
 			(at 67.818 162.56 0)
 			(show_name no)
@@
 			)
 		)
-		(property "Value" "10u"
+		(property "Value" "1u"
 			(at 146.558 100.33 0)
 			(show_name no)
@@
 			)
 		)
-		(property "Value" "0.47uH"
+		(property "Value" "0.47u"
 			(at 120.65 98.298 90)
 			(show_name no)
@@
 			)
 		)
-		(property "Value" "10u"
+		(property "Value" "1u"
 			(at 146.558 115.57 0)
 			(show_name no)
@@
 			)
 		)
-		(property "Value" "10u"
+		(property "Value" "1u"
 			(at 259.588 129.54 0)
 			(show_name no)
@@
 			)
 		)
-		(property "Value" "10u"
+		(property "Value" "1u"
 			(at 137.668 100.33 0)
 			(show_name no)
@@
 			)
 		)
-		(property "Value" "100n"
+		(property "Value" "1u"
 			(at 216.408 34.29 0)
 			(show_name no)
@@
 			)
 		)
-		(property "Value" "10u"
+		(property "Value" "1u"
 			(at 103.378 43.18 0)
 			(show_name no)
@@
 			)
 		)
-		(property "Value" "10u"
+		(property "Value" "1u"
 			(at 57.658 100.33 0)
 			(show_name no)
@@
 			)
 		)
-		(property "Value" "10u"
+		(property "Value" "1u"
 			(at 67.818 100.33 0)
 			(show_name no)
@@
 			)
 		)
-		(property "Value" "10u"
+		(property "Value" "1u"
 			(at 137.668 115.57 0)
 			(show_name no)

Commit message: Fix small errors for the design
Parts:
- removed J_BATT301: S2B-PH-SM4-TB, Connector_JST:JST_PH_S2B-PH-SM4-TB_1x02-1MP_P2.00mm_Horizontal, symbol S2B_PH_SM4_TB:S2B-PH-SM4-TB
- added J_BATT301: S2B-PH-SM4-TB, connectors:JST_PH_S2B-PH-SM4-TB_1x02-1MP_P2.00mm_Horizontal, symbol connectors:S2B-PH-SM4-TB
- renumbered C308 to C301, C310 to C302, C309 to C303, C311 to C304, C312 to C305, C313 to C306, C314 to C307, C301 to C308, C302 to C309, C315 to C310, C316 to C311, C317 to C312, C318 to C313, C319 to C314, C320 to C315, C303 to C316, C305 to C317, C307 to C318, C321 to C319, C304 to C320, C306 to C321, R303 to R301, R301 to R302, R302 to R303
Connections:
- net GND: now also J_BATT301.2, J_BATT301.MP (SHIELD)
- net at C318.1, U301.C2 (BAT): now also J_BATT301.1
